Commit message: Velodyne with gpu acceleration

File: src/jackal_description/urdf/accessories.urdf.xacro (robot description, xacro)
@@ -176,7 +176,8 @@
     <xacro:property name="parent" value="$(optenv JACKAL_LASER_3D_PARENT ${mount}_mount)" />
     <xacro:property name="lidar_3d_model" value="$(optenv JACKAL_LASER_3D_MODEL vlp16)" />
+    <!-- <xacro:property name="gpu" value="true" /> -->
     <!-- Velodyne VLP16 -->
     <xacro:if value="${lidar_3d_model == 'vlp16'}">
-      <xacro:vlp16_mount topic="${topic}" tower="${tower}" prefix="${prefix}" parent_link="${parent}" >
+      <xacro:vlp16_mount topic="${topic}" tower="${tower}" prefix="${prefix}" parent_link="${parent}">
         <origin xyz="$(optenv JACKAL_LASER_3D_OFFSET 0 0 0)" rpy="$(optenv JACKAL_LASER_3D_RPY 0 0 0)" />
       </xacro:vlp16_mount>

File: src/jackal_description/urdf/accessories/vlp16_mount.urdf.xacro (robot description, xacro)
@@ -1,5 +1,5 @@
 <robot xmlns:xacro="http://wiki.ros.org/xacro">
   <xacro:include filename="$(find velodyne_description)/urdf/VLP-16.urdf.xacro" />
-  <xacro:macro name="vlp16_mount" params="prefix parent_link topic tower height:=0.1 *origin">
+  <xacro:macro name="vlp16_mount" params="prefix parent_link topic tower height:=0.1 *origin gpu:=true">
     <xacro:if value="${tower}">
       <link name="${prefix}_vlp16_mount" />

Commit message: Added kinect to jackal

File: src/jackal_description/urdf/accessories.urdf.xacro (robot description, xacro)
@@ -52,5 +52,5 @@
     <xacro:property name="prefix" value="$(optenv JACKAL_LASER_PREFIX ${mount})" />
     <xacro:property name="parent" value="$(optenv JACKAL_LASER_PARENT ${mount}_mount)" />
-    <xacro:property name="lidar_model" value="$(optenv JACKAL_LASER_MODEL tim551)" />
+    <xacro:property name="lidar_model" value="$(optenv JACKAL_LASER_MODEL utm30)" />
     <xacro:property name="mount_type" value="$(optenv JACKAL_LASER_MOUNT_TYPE upright)" />
     <!-- SICK LMS1xx -->
@@ -104,10 +104,10 @@
     <xacro:if value="${lidar_model == 'utm30'}">
       <xacro:hokuyo_utm30_mount topic="${topic}" prefix="${prefix}" parent_link="${parent}">
-        <origin xyz="$(optenv JACKAL_LASER_OFFSET 0 0 0)" rpy="$(optenv JACKAL_LASER_RPY 0 0 0)" />
+        <origin xyz="$(optenv JACKAL_LASER_OFFSET 0.12 0 -0.18)" rpy="$(optenv JACKAL_LASER_RPY 0 0 0)" />
       </xacro:hokuyo_utm30_mount>
     </xacro:if>
   </xacro:if>
   <!-- Secondary 2D Lidar -->
-  <xacro:if value="$(optenv JACKAL_LASER_SECONDARY 0)">
+  <xacro:if value="$(optenv JACKAL_LASER_SECONDARY 1)">
     <xacro:property name="mount" value="$(optenv JACKAL_LASER_SECONDARY_MOUNT rear)" />
     <xacro:property name="topic" value="$(optenv JACKAL_LASER_SECONDARY_TOPIC rear/scan)" />
@@ -116,11 +116,19 @@
     <xacro:property name="parent" value="$(optenv JACKAL_LASER_SECONDARY_PARENT ${mount}_mount)" />
     <xacro:property name="lidar_model" value="$(optenv JACKAL_LASER_SECONDARY_MODEL lms1xx)" />
+    <xacro:property name="mount_type" value="$(optenv JACKAL_LASER_MOUNT_TYPE upright)" />
     <!-- SICK LMS1xx -->
     <xacro:if value="${lidar_model == 'lms1xx'}">
       <!-- Mount Enabled -->
       <xacro:if value="${tower}">
-        <xacro:sick_lms1xx_mount topic="${topic}" prefix="${prefix}" parent_link="${parent}">
-          <origin xyz="$(optenv JACKAL_LASER_SECONDARY_OFFSET 0 0 0)" rpy="$(optenv JACKAL_LASER_SECONDARY_RPY 0 0 3.14159)" />
-        </xacro:sick_lms1xx_mount>
+       <xacro:if value="${mount_type == 'upright'}">
+        <xacro:sick_lms1xx_upright_mount topic="${topic}" prefix="${prefix}" parent_link="${parent}">
+          <origin xyz="$(optenv JACKAL_LASER_SECONDARY_OFFSET 0 0 0)" rpy="$(optenv JACKAL_LASER_SECONDARY_RPY 0 0 0)" />
+        </xacro:sick_lms1xx_upright_mount>
+       </xacro:if>
+       <xacro:if value="${mount_type == 'inverted'}">
+      	 <xacro:sick_lms1xx_inverted_mount topic="${topic}" prefix="${prefix}" parent_link="${parent}">
+           <origin xyz="$(optenv JACKAL_LASER_OFFSET 0 0 0)" rpy="$(optenv JACKAL_LASER_RPY 0 0 0)" />
+         </xacro:sick_lms1xx_inverted_mount>
+       </xacro:if>
       </xacro:if>
       <!-- Mount Disabled -->
@@ -176,8 +184,7 @@
     <xacro:property name="parent" value="$(optenv JACKAL_LASER_3D_PARENT ${mount}_mount)" />
     <xacro:property name="lidar_3d_model" value="$(optenv JACKAL_LASER_3D_MODEL vlp16)" />
-    <!-- <xacro:property name="gpu" value="true" /> -->
     <!-- Velodyne VLP16 -->
     <xacro:if value="${lidar_3d_model == 'vlp16'}">
-      <xacro:vlp16_mount topic="${topic}" tower="${tower}" prefix="${prefix}" parent_link="${parent}">
+      <xacro:vlp16_mount topic="${topic}" tower="${tower}" prefix="${prefix}" parent_link="${parent}" >
         <origin xyz="$(optenv JACKAL_LASER_3D_OFFSET 0 0 0)" rpy="$(optenv JACKAL_LASER_3D_RPY 0 0 0)" />
       </xacro:vlp16_mount>
@@ -261,5 +268,5 @@
   <xacro:include filename="$(find pointgrey_camera_description)/urdf/pointgrey_flea3.urdf.xacro" />
   <!-- If enabled, generate the flea3 camera payload with a tilt of 30 degrees. -->
-  <xacro:if value="$(optenv JACKAL_FLEA3 1)">
+  <xacro:if value="$(optenv JACKAL_FLEA3 0)">
     <xacro:property name="name" value="$(optenv JACKAL_FLEA3_NAME front)" />
     <xacro:property name="tilt" value="$(optenv JACKAL_FLEA3_TILT 0.)" />

File: src/jackal_description/urdf/accessories/hokuyo_utm30.urdf.xacro (robot description, xacro)
@@ -3,5 +3,5 @@
   <xacro:macro name="hokuyo_utm30_mount" params="prefix topic parent_link min_angle:=-2.2689  max_angle:=2.2689 *origin">
     <xacro:macro name="hokuyo_utm30" params="frame:=laser topic:=scan sample_size:=1440 update_rate:=50
-               min_angle:=-2.2689 max_angle:=2.2689 min_range:=0.1 max_range:=30.0 robot_namespace:=/">
+               min_angle:=-1.5708 max_angle:=1.5708 min_range:=0.1 max_range:=30.0 robot_namespace:=/">
       <xacro:property name="mass" value="0.370"/>
       <xacro:property name="base" value="0.06" />

File: src/jackal_description/urdf/accessories/sick_lms1xx_upright_mount.urdf.xacro (robot description, xacro)
@@ -36,20 +36,33 @@
     <link name="${prefix}_laser_mount">
       <visual>
-        <origin xyz="0 0 0" rpy="0 0 0" />
-        <geometry>
-          <!-- Origin of this mesh is the base of the bracket. -->
-          <mesh filename="package://jackal_description/meshes/sick-lms1xx-upright-bracket.stl" />
-        </geometry>
-        <material name="dark_grey" />
-      </visual>
+          <geometry>
+            <cylinder radius="0.055" length = "0.42"/>
+          </geometry>
+          <origin xyz="0 0 0" rpy="0 0 0" />
+          <material name="white" />
+        </visual>
+        <collision>
+          <geometry>
+            <cylinder radius="0.055" length = "0.42"/>
+          </geometry>
+          <origin xyz="0 0 0" rpy="0 0 0" />
+        </collision>
+        <inertial>
+          <origin xyz="0 0 0" rpy="0 0 0"/>
+          <mass value="0.2"/>
+          <inertia
+            ixx="0.0012779167" ixy="0" ixz="0"
+            iyy="0.0012779167" iyz="0"
+            izz="0.0003025"/>
+        </inertial>
     </link>
     <joint name="${prefix}_laser_joint" type="fixed">
       <!-- This offset is from the base of the bracket to the LIDAR's focal point. -->
-      <origin xyz="0 0 0.149" rpy="0 0 0" />
+      <origin xyz="0 0 0.3256" rpy="0 0 0" />
       <parent link="${prefix}_laser_mount" />
       <child link="${prefix}_laser" />
     </joint>
     <gazebo reference="${prefix}_laser_mount">
-      <material>Gazebo/DarkGrey</material>
+      <material>Gazebo/White</material>
     </gazebo>
   </xacro:macro>

File: src/jackal_description/urdf/accessories/vlp16_mount.urdf.xacro (robot description, xacro)
@@ -1,5 +1,5 @@
 <robot xmlns:xacro="http://wiki.ros.org/xacro">
   <xacro:include filename="$(find velodyne_description)/urdf/VLP-16.urdf.xacro" />
-  <xacro:macro name="vlp16_mount" params="prefix parent_link topic tower height:=0.1 *origin gpu:=true">
+  <xacro:macro name="vlp16_mount" params="prefix parent_link topic tower height:=0.1 *origin">
     <xacro:if value="${tower}">
       <link name="${prefix}_vlp16_mount" />

File: src/jackal_description/urdf/jackal.urdf.xacro (robot description, xacro)
@@ -218,4 +218,12 @@
     <origin xyz="${mount_spacing} 0 0" />
   </joint>
+  <!-- add depth camera to the chassis -->
+  <xacro:include filename="$(find jackal_description)/urdf/kinect_camera.xacro" />
+  <xacro:kinect_camera prefix="kinect"/>
+  <joint name="kinect_joint" type="fixed">
+    <parent link="mid_mount" />
+    <child link="kinect_link" />
+    <origin xyz="0.15 0 0.035" />
+  </joint>
   <!-- Bring in simulation data for Gazebo. -->
   <xacro:include filename="$(find jackal_description)/urdf/jackal.gazebo" />
